Commit message: implemented task 7A.1 and 7A.2 and tested both of them

File: Rover/my_robot_description/urdf/my_robot.urdf.xacro (robot description, xacro)
@@ -79,11 +79,10 @@
     <!-- Empty link - just a reference frame -->
   </link>
-  <!-- Joint connecting footprint to base_link -->
-  <!-- Z offset calculated to place base above ground with wheels touching -->
+  <!-- Joint connecting base_link to footprint (ground reference) -->
   <joint name="base_footprint_joint" type="fixed">
-    <parent link="${base_footprint_name}"/>
-    <child link="${base_link_name}"/>
-    <!-- Height = base_height/2 + arm_height + wheel_radius -->
-    <origin xyz="0 0 ${base_height/2 + arm_height + wheel_radius}" rpy="0 0 0"/>
+    <parent link="${base_link_name}"/>
+    <child link="${base_footprint_name}"/>
+    <!-- Ground level below base_link center -->
+    <origin xyz="0 0 ${-(base_height/2 + arm_height + wheel_radius)}" rpy="0 0 0"/>
   </joint>
   <!-- ========================================== -->
