Commit message: editing the docker container and also editing the rover model solving TF tree proplems

File: Rover/my_robot_description/urdf/gazebo.xacro (robot description, xacro)
@@ -103,5 +103,5 @@
       <odom_publish_frequency>50</odom_publish_frequency>
       <odom_topic>odom</odom_topic>
-      <tf_topic>tf</tf_topic>
+      <tf_topic>/model/my_robot/tf</tf_topic>
       <!-- Frame IDs -->
       <frame_id>odom</frame_id>

File: Rover/my_robot_description/urdf/my_robot.urdf.xacro (robot description, xacro)
@@ -79,10 +79,10 @@
     <!-- Empty link - just a reference frame -->
   </link>
-  <!-- Joint connecting base_link to footprint (ground reference) -->
+  <!-- Joint connecting footprint (ground reference) to base_link (chassis) -->
   <joint name="base_footprint_joint" type="fixed">
-    <parent link="${base_link_name}"/>
-    <child link="${base_footprint_name}"/>
-    <!-- Ground level below base_link center -->
-    <origin xyz="0 0 ${-(base_height/2 + arm_height + wheel_radius)}" rpy="0 0 0"/>
+    <parent link="${base_footprint_name}"/>
+    <child link="${base_link_name}"/>
+    <!-- Height of base_link center above ground -->
+    <origin xyz="0 0 ${base_height/2 + arm_height + wheel_radius}" rpy="0 0 0"/>
   </joint>
   <!-- ========================================== -->

Commit message: editing the rover model and changing what is needed for it be work ( still needs validation )

File: Rover/my_robot_description/urdf/gazebo.xacro (robot description, xacro)
@@ -18,14 +18,8 @@
     <material>Gazebo/Grey</material>
   </gazebo>
-  <gazebo reference="left_middle_arm_link">
-    <material>Gazebo/Grey</material>
-  </gazebo>
   <gazebo reference="left_rear_arm_link">
     <material>Gazebo/Grey</material>
   </gazebo>
   <gazebo reference="right_front_arm_link">
-    <material>Gazebo/Grey</material>
-  </gazebo>
-  <gazebo reference="right_middle_arm_link">
     <material>Gazebo/Grey</material>
   </gazebo>
@@ -36,11 +30,4 @@
   <!-- High friction for wheels, low damping for smooth rolling -->
   <gazebo reference="left_front_wheel_link">
-    <material>Gazebo/Black</material>
-    <mu1>1.0</mu1>
-    <mu2>1.0</mu2>
-    <kp>1000000.0</kp>
-    <kd>1.0</kd>
-  </gazebo>
-  <gazebo reference="left_middle_wheel_link">
     <material>Gazebo/Black</material>
     <mu1>1.0</mu1>
@@ -63,11 +50,4 @@
     <kd>1.0</kd>
   </gazebo>
-  <gazebo reference="right_middle_wheel_link">
-    <material>Gazebo/Black</material>
-    <mu1>1.0</mu1>
-    <mu2>1.0</mu2>
-    <kp>1000000.0</kp>
-    <kd>1.0</kd>
-  </gazebo>
   <gazebo reference="right_rear_wheel_link">
     <material>Gazebo/Black</material>
@@ -79,13 +59,11 @@
   <!-- Differential Drive Plugin for Gazebo (ROS 2 Jazzy) -->
   <!-- This plugin allows controlling the robot using /cmd_vel topic -->
-  <!-- It simulates a 6-wheel skid-steer rover -->
+  <!-- It simulates a 4-wheel tank-style skid-steer rover -->
   <gazebo>
     <plugin filename="gz-sim-diff-drive-system" name="gz::sim::systems::DiffDrive">
-      <!-- Wheel joints to control (all 6 wheels for skid-steer drive) -->
+      <!-- Wheel joints to control (4 wheels for 4WD tank-style skid-steer drive) -->
       <left_joint>left_front_wheel_joint</left_joint>
-      <left_joint>left_middle_wheel_joint</left_joint>
       <left_joint>left_rear_wheel_joint</left_joint>
       <right_joint>right_front_wheel_joint</right_joint>
-      <right_joint>right_middle_wheel_joint</right_joint>
       <right_joint>right_rear_wheel_joint</right_joint>
       <!-- Wheel separation and diameter -->

File: Rover/my_robot_description/urdf/my_robot.urdf.xacro (robot description, xacro)
@@ -2,7 +2,7 @@
 <!--
   my_robot.urdf.xacro - Mars Rover Style Robot Description
-  This file defines a 6-wheeled Mars rover style robot with:
+  This file defines a 4-wheeled Mars rover style robot with:
   - Square base (0.4m × 0.4m × 0.15m) in RED color
-  - 6 wheels: 3 on left side, 3 on right side
+  - 4 wheels: 2 on left side, 2 on right side (4WD tank-style skid-steer)
   - Each wheel connected via continuous joint for driving
   The robot uses xacro macros for reusability and maintainability.
@@ -44,5 +44,5 @@
   <!--
     TO SHIFT SUSPENSION ARMS AND WHEELS:
-    - Edit wheel_x_front, wheel_x_middle, wheel_x_rear to move wheels forward/backward
+    - Edit wheel_x_front, wheel_x_rear to move wheels forward/backward
     - Edit arm_y_offset to move arms (and wheels) left/right
     - Edit arm_x_offset to move arms forward/backward relative to wheels
@@ -55,7 +55,6 @@
   <!-- Y offset: arms extend from sides of base (outside the base body) -->
   <xacro:property name="arm_y_offset" value="0.21"/>
-  <!-- X positions: front, middle, rear (evenly spaced along base length) -->
+  <!-- X positions: front and rear for 4-wheel rover -->
   <xacro:property name="wheel_x_front" value="0.15"/>
-  <xacro:property name="wheel_x_middle" value="0.0"/>
   <xacro:property name="wheel_x_rear" value="-0.15"/>
   <!-- Wheel offset relative to arm link (fine-tune wheel position) -->
@@ -109,17 +108,11 @@
   </link>
   <!-- ========================================== -->
-  <!-- SUSPENSION ARMS + WHEELS (Mars rover style) -->
-  <!-- 6 rectangular arms extending down from base -->
-  <!-- 6 wheels attached to bottom of arms         -->
+  <!-- SUSPENSION ARMS + WHEELS (4-Wheel Tank Drive) -->
+  <!-- 4 rectangular arms extending down from base -->
+  <!-- 4 wheels attached to bottom of arms         -->
   <!-- ========================================== -->
   <!-- LEFT SIDE -->
   <xacro:suspension_wheel_macro prefix="left_front"
                                 x_pos="${wheel_x_front}"
-                                y_pos="${arm_y_offset}"
-                                wheel_offset_x="${wheel_offset_x_left}"
-                                wheel_offset_y="${wheel_offset_y_left}"
-                                wheel_offset_z="${wheel_offset_z_left}"/>
-  <xacro:suspension_wheel_macro prefix="left_middle"
-                                x_pos="${wheel_x_middle}"
                                 y_pos="${arm_y_offset}"
                                 wheel_offset_x="${wheel_offset_x_left}"
@@ -139,10 +132,4 @@
                                 wheel_offset_y="${wheel_offset_y_right}"
                                 wheel_offset_z="${wheel_offset_z_right}"/>
-  <xacro:suspension_wheel_macro prefix="right_middle"
-                                x_pos="${wheel_x_middle}"
-                                y_pos="${-arm_y_offset}"
-                                wheel_offset_x="${wheel_offset_x_right}"
-                                wheel_offset_y="${wheel_offset_y_right}"
-                                wheel_offset_z="${wheel_offset_z_right}"/>
   <xacro:suspension_wheel_macro prefix="right_rear"
                                 x_pos="${wheel_x_rear}"

Commit message: refactor(rover): convert rover model and simulation from 6-wheel to 4-wheel configuration
- Remove middle wheels and arms from URDF (my_robot.urdf.xacro, macros.xacro)
- Update Gazebo DiffDrive plugin in gazebo.xacro to 4 joints
- Configure encoder_ticks_to_odom.py for 4-wheel kinematics and URDF joint matching
- Add unit and regression tests for 4-wheel joint matching (39 passing)
- Remove middle link references from RViz config files
- Add .agents/ to .gitignore

File: Rover/my_robot_description/urdf/gazebo.xacro (robot description, xacro)
@@ -18,14 +18,8 @@
     <material>Gazebo/Grey</material>
   </gazebo>
-  <gazebo reference="left_middle_arm_link">
-    <material>Gazebo/Grey</material>
-  </gazebo>
   <gazebo reference="left_rear_arm_link">
     <material>Gazebo/Grey</material>
   </gazebo>
   <gazebo reference="right_front_arm_link">
-    <material>Gazebo/Grey</material>
-  </gazebo>
-  <gazebo reference="right_middle_arm_link">
     <material>Gazebo/Grey</material>
   </gazebo>
@@ -36,11 +30,4 @@
   <!-- High friction for wheels, low damping for smooth rolling -->
   <gazebo reference="left_front_wheel_link">
-    <material>Gazebo/Black</material>
-    <mu1>1.0</mu1>
-    <mu2>1.0</mu2>
-    <kp>1000000.0</kp>
-    <kd>1.0</kd>
-  </gazebo>
-  <gazebo reference="left_middle_wheel_link">
     <material>Gazebo/Black</material>
     <mu1>1.0</mu1>
@@ -63,11 +50,4 @@
     <kd>1.0</kd>
   </gazebo>
-  <gazebo reference="right_middle_wheel_link">
-    <material>Gazebo/Black</material>
-    <mu1>1.0</mu1>
-    <mu2>1.0</mu2>
-    <kp>1000000.0</kp>
-    <kd>1.0</kd>
-  </gazebo>
   <gazebo reference="right_rear_wheel_link">
     <material>Gazebo/Black</material>
@@ -79,13 +59,11 @@
   <!-- Differential Drive Plugin for Gazebo (ROS 2 Jazzy) -->
   <!-- This plugin allows controlling the robot using /cmd_vel topic -->
-  <!-- It simulates a 6-wheel skid-steer rover -->
+  <!-- It simulates a 4-wheel skid-steer rover -->
   <gazebo>
     <plugin filename="gz-sim-diff-drive-system" name="gz::sim::systems::DiffDrive">
-      <!-- Wheel joints to control (all 6 wheels for skid-steer drive) -->
+      <!-- Wheel joints to control (4 wheels for skid-steer drive) -->
       <left_joint>left_front_wheel_joint</left_joint>
-      <left_joint>left_middle_wheel_joint</left_joint>
       <left_joint>left_rear_wheel_joint</left_joint>
       <right_joint>right_front_wheel_joint</right_joint>
-      <right_joint>right_middle_wheel_joint</right_joint>
       <right_joint>right_rear_wheel_joint</right_joint>
       <!-- Wheel separation and diameter -->

File: Rover/my_robot_description/urdf/macros.xacro (robot description, xacro)
@@ -76,5 +76,5 @@
     Arm connects vertically through wheel CENTER
     Parameters:
-      prefix - identifier (e.g., "left_front", "right_middle")
+      prefix - identifier (e.g., "left_front", "right_rear")
       x_pos - x position relative to base_link (m)
       y_pos - y position relative to base_link (m)

File: Rover/my_robot_description/urdf/my_robot.urdf.xacro (robot description, xacro)
@@ -2,7 +2,7 @@
 <!--
   my_robot.urdf.xacro - Mars Rover Style Robot Description
-  This file defines a 6-wheeled Mars rover style robot with:
+  This file defines a 4-wheeled Mars rover style robot with:
   - Square base (0.4m × 0.4m × 0.15m) in RED color
-  - 6 wheels: 3 on left side, 3 on right side
+  - 4 wheels: 2 on left side, 2 on right side
   - Each wheel connected via continuous joint for driving
   The robot uses xacro macros for reusability and maintainability.
@@ -44,5 +44,5 @@
   <!--
     TO SHIFT SUSPENSION ARMS AND WHEELS:
-    - Edit wheel_x_front, wheel_x_middle, wheel_x_rear to move wheels forward/backward
+    - Edit wheel_x_front, wheel_x_rear to move wheels forward/backward
     - Edit arm_y_offset to move arms (and wheels) left/right
     - Edit arm_x_offset to move arms forward/backward relative to wheels
@@ -55,7 +55,6 @@
   <!-- Y offset: arms extend from sides of base (outside the base body) -->
   <xacro:property name="arm_y_offset" value="0.21"/>
-  <!-- X positions: front, middle, rear (evenly spaced along base length) -->
+  <!-- X positions: front, rear (+0.15m and -0.15m along base length) -->
   <xacro:property name="wheel_x_front" value="0.15"/>
-  <xacro:property name="wheel_x_middle" value="0.0"/>
   <xacro:property name="wheel_x_rear" value="-0.15"/>
   <!-- Wheel offset relative to arm link (fine-tune wheel position) -->
@@ -110,16 +109,10 @@
   <!-- ========================================== -->
   <!-- SUSPENSION ARMS + WHEELS (Mars rover style) -->
-  <!-- 6 rectangular arms extending down from base -->
-  <!-- 6 wheels attached to bottom of arms         -->
+  <!-- 4 rectangular arms extending down from base -->
+  <!-- 4 wheels attached to bottom of arms         -->
   <!-- ========================================== -->
   <!-- LEFT SIDE -->
   <xacro:suspension_wheel_macro prefix="left_front"
                                 x_pos="${wheel_x_front}"
-                                y_pos="${arm_y_offset}"
-                                wheel_offset_x="${wheel_offset_x_left}"
-                                wheel_offset_y="${wheel_offset_y_left}"
-                                wheel_offset_z="${wheel_offset_z_left}"/>
-  <xacro:suspension_wheel_macro prefix="left_middle"
-                                x_pos="${wheel_x_middle}"
                                 y_pos="${arm_y_offset}"
                                 wheel_offset_x="${wheel_offset_x_left}"
@@ -139,10 +132,4 @@
                                 wheel_offset_y="${wheel_offset_y_right}"
                                 wheel_offset_z="${wheel_offset_z_right}"/>
-  <xacro:suspension_wheel_macro prefix="right_middle"
-                                x_pos="${wheel_x_middle}"
-                                y_pos="${-arm_y_offset}"
-                                wheel_offset_x="${wheel_offset_x_right}"
-                                wheel_offset_y="${wheel_offset_y_right}"
-                                wheel_offset_z="${wheel_offset_z_right}"/>
   <xacro:suspension_wheel_macro prefix="right_rear"
                                 x_pos="${wheel_x_rear}"
